File: Keyboard-PCB V1.0.kicad_sch (KiCad schematic)
At the start: 24 parts, among them U1 ATmega32U4-A

Commit message: Footprints Added
Parts:
- MX1, MX2, MX3, MX4: footprint (none) -> MX_Hotswap:MX-Hotswap-1U
- Polyfuse1: footprint (none) -> Fuse:Fuse_1206_3216Metric
- R_D+1, R_D-1, R_PE2, R_pull_up1: footprint (none) -> Resistor_SMD:R_0805_2012Metric
- Switch1: footprint (none) -> random-keyboard-parts:SKQG-1155865
Other:
- title: (none) -> Mechanical Keyboard PCB V1.0
Changed lines of the file:
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@@
 	(generator_version "8.0")
 	(paper "A4")
+	(title_block
+		(title "Mechanical Keyboard PCB V1.0")
+		(date "2024-08-16")
+	)
 	(junction
 		(at 146.685 91.44)
@@
 			)
 		)
-		(property "Footprint" ""
+		(property "Footprint" "MX_Hotswap:MX-Hotswap-1U"
 			(at 136.525 83.185 0)
 			(effects
@@
 			)
 		)
-		(property "Footprint" ""
+		(property "Footprint" "Resistor_SMD:R_0805_2012Metric"
 			(at 59.69 85.09 0)
 			(effects
@@
 			)
 		)
-		(property "Footprint" ""
+		(property "Footprint" "random-keyboard-parts:SKQG-1155865"
 			(at 52.705 48.26 0)
 			(effects
@@
 			)
 		)
-		(property "Footprint" ""
+		(property "Footprint" "Fuse:Fuse_1206_3216Metric"
 			(at 67.945 167.64 0)
 			(effects
@@
 			)
 		)
-		(property "Footprint" ""
+		(property "Footprint" "MX_Hotswap:MX-Hotswap-1U"
 			(at 154.305 64.135 0)
 			(effects
@@
 			)
 		)
-		(property "Footprint" ""
+		(property "Footprint" "Resistor_SMD:R_0805_2012Metric"
 			(at 69.215 87.63 0)
 			(effects
@@
 			)
 		)
-		(property "Footprint" ""
+		(property "Footprint" "MX_Hotswap:MX-Hotswap-1U"
 			(at 136.525 64.135 0)
 			(effects
@@
 			)
 		)
-		(property "Footprint" ""
+		(property "Footprint" "MX_Hotswap:MX-Hotswap-1U"
 			(at 154.305 83.185 0)
 			(effects
@@
 			)
 		)
-		(property "Footprint" ""
+		(property "Footprint" "Resistor_SMD:R_0805_2012Metric"
 			(at 65.405 43.815 0)
 			(effects
@@
 			)
 		)
-		(property "Footprint" ""
+		(property "Footprint" "Resistor_SMD:R_0805_2012Metric"
 			(at 118.745 113.03 0)
 			(effects
